Commit message: Puzzlebot se ve bien

File: urdf/puzzlebot_jetson_ed_urdf.urdf (robot description, URDF)
Before this commit: robot Puzzlebot Jetson-Lidar Ed., 4 links, 3 joints
Links:
- link wl_link: mass None -> 0.03
Joints:
- joint leftWheel: origin xyz=0.05 0.0955 0 -> xyz=0.05 0.0955 0.05 rpy=0 0 0
- joint rightWheel: origin xyz=0.05 -0.0955 0 -> xyz=0.05 -0.0955 0.05 rpy=0 0 0; parent chassis -> base_link

Commit message: animacion

File: urdf/puzzlebot_jetson_ed_urdf.urdf (robot description, URDF)
Before this commit: robot Puzzlebot Jetson-Lidar Ed., 4 links, 3 joints
Joints:
- joint rightWheel: parent base_link -> chassis
